File: EVM_741_signal_routing.kicad_pcb (KiCad board)
At the start: 2 copper layers, 80 x 50.2 mm, 49 parts, among them J1 offset+, J10 out_a, J11 out_j, J12 out_j, J13 Vcc+_a, J14 Vcc-_a, J2 in-, J3 in+, J4 Vcc-, J5 offset-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

Commit message: fixed silkscreen
Parts:
- J1: value offset+ -> off+
- J10: value out_a -> out
- J5: value offset- -> off-
- J8: value in+_a -> in+
- J9: value in-_a -> in-
- turned J2 to 180 degrees
- turned J5 to 180 degrees
- turned J9 to 180 degrees
Connections:
- net vin_sine renamed Net-(J3-Pin_1)
